File: PCB/V1/V1.kicad_pcb (KiCad board)
At the start: 2 copper layers, 100 x 100 mm, 19 parts, among them J1 Bornera Motores, J2 Bateria2, J3 Bateria1, SW1 SW ON/OFF MOTORES, SW2 SW 24V/12V, SW3 SW ON/OFF, U1 ESP32-Devkit-V1

Commit message: .
Parts:
- removed the ? at (202.9, 111.7)
- added ?: , , F.Cu at (219.2, 37.8)
- added ?: , , F.Cu at (132.1, 130.7)
- added R4: 10K, Resistor_THT:R_Axial_DIN0207_L6.3mm_D2.5mm_P10.16mm_Horizontal, F.Cu at (192.9, 128.0)
- added SW4: SW_Push, TerminalBlock:TerminalBlock_bornier-2_P5.08mm, F.Cu at (214.0, 130.5)
- D5: footprint LED_THT:LED_D5.0mm_Horizontal_O1.27mm_Z3.0mm -> Connector_Molex:Molex_KK-254_AE-6410-02A_1x02_P2.54mm_Vertical; moved to F.Cu
- moved D5 13.2 mm to (207.0, 106.5)
Connections:
- U1 pad 3: unconnected-(U1-IO13-Pad3) -> BTN1
- U1 pad 30: unconnected-(U1-3v3-Pad30) -> +3V3
Routing:
- net +3V3: track 0.00 -> 64.3 mm, vias 0 -> 2
- net BTN1: track 0.00 -> 39.8 mm
- net GND: track 275.9 -> 312.5 mm
- net LED BLUETOOTH: track 23.5 -> 40.1 mm
- net Net-(D5-K): track 3.81 -> 13.6 mm
- net Net-(SW2A-B): track 28.7 -> 19.0 mm
Other:
- board size 100 x 100 mm -> 100 x 101 mm

Commit message: .
Parts:
- removed J2: Bateria2, Connector_AMASS:AMASS_XT60-M_1x02_P7.20mm_Vertical
- removed SW2: SW 24V/12V, Button_Switch_THT:SW_Slide_SPDT_Angled_CK_OS102011MA1Q
- R3: value 47 -> 87
- SW3: footprint Button_Switch_THT:SW_Slide_SPDT_Angled_CK_OS102011MA1Q -> TerminalBlock:TerminalBlock_bornier-2_P5.08mm
- moved D4 112.6 mm to (132.2, 132.1), turned to 0 degrees
- moved R2 107.6 mm to (131.7, 127.6), turned to 90 degrees
- moved ? 87.7 mm to (143.1, 43.7)
- moved ? 79.8 mm to (217.4, 117.6)
- moved SW3 45.1 mm to (132.9, 67.7), turned to 90 degrees
- moved J3 14.4 mm to (133.4, 44.8), turned to -90 degrees
- moved J1 4.54 mm to (216.6, 45.7)
Connections:
- SW3 pad 1: Net-(SW2A-B) -> GND
Routing:
- net GND: track 312.5 -> 404.4 mm
- net LED ON/OFF: track 205.7 -> 175.7 mm
- net Net-(SW2A-B): track 19.0 -> 0.00 mm
- net Net-(J2-Pin_1): track 16.4 -> 0.00 mm
- net Net-(D1-A): track 53.1 -> 38.3 mm
- net Net-(J3-Pin_2): track 20.9 -> 10.8 mm
- net Net-(D4-K): track 3.15 -> 4.66 mm
Other:
- board size 100 x 101 mm -> 100 x 98.9 mm
- board text added: "IN+"

Commit message: .
Parts:
- moved SW1 8.90 mm to (218.4, 84.1)
Routing:
- net Led Monster: track 77.2 -> 71.5 mm
- net +5V: track 218.1 -> 223.6 mm
- net GND: track 404.4 -> 405.9 mm
- net BTN1: track 39.8 -> 40.5 mm
Changed lines of the file:
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@@
 		(tags "LED diameter 5.0mm z-position of LED center 3.0mm 2 pins")
 		(property "Reference" "D4"
-			(at 1.27 -1.96 360)
+			(at 1.27 -1.96 0)
 			(layer "F.SilkS")
 			(effects
@@
 		)
 		(property "Value" "LED ON/OFF"
-			(at 1.27 10.93 360)
+			(at 1.27 10.93 0)
 			(layer "F.Fab")
 			(effects
@@
 	(footprint "Button_Switch_THT:SW_Slide_SPDT_Angled_CK_OS102011MA1Q"
 		(layer "F.Cu")
-		(at 209.55 84.55 90)
+		(at 218.44 84.09 90)
 		(descr "CuK miniature slide switch, OS series, SPDT, right angle, http://www.ckswitches.com/media/1428/os.pdf")
 		(tags "switch SPDT")
@@
 	)
 	(segment
-		(start 209.55 82.55)
-		(end 213.36 82.55)
+		(start 221.19 67.52)
+		(end 210.82 57.15)
 		(width 1)
 		(layer "B.Cu")
@@
 	)
 	(segment
-		(start 210.82 57.15)
-		(end 179.07 57.15)
+		(start 162.56 57.15)
+		(end 161.925 56.515)
 		(width 1)
 		(layer "B.Cu")
@@
 	)
 	(segment
-		(start 162.56 57.15)
-		(end 161.925 56.515)
+		(start 212.09 115.57)
+		(end 207.01 115.57)
 		(width 1)
 		(layer "B.Cu")
@@
 	)
 	(segment
-		(start 213.36 82.55)
-		(end 213.36 59.69)
+		(start 221.19 82.84)
+		(end 221.19 106.47)
 		(width 1)
 		(layer "B.Cu")
@@
 	)
 	(segment
-		(start 212.09 115.57)
-		(end 207.01 115.57)
+		(start 220.44 82.09)
+		(end 220.83 82.48)
+		(width 1)
+		(layer "B.Cu")
+		(net 7)
+	)
+	(segment
+		(start 221.19 106.47)
+		(end 212.09 115.57)
 		(width 1)
 		(layer "B.Cu")
@@
 	)
 	(segment
-		(start 187.325 123.19)
-		(end 187.325 130.81)
+		(start 220.83 82.48)
+		(end 221.19 82.12)
 		(width 1)
 		(layer "B.Cu")
@@
 	)
 	(segment
-		(start 213.36 59.69)
-		(end 210.82 57.15)
+		(start 187.325 123.19)
+		(end 187.325 130.81)
 		(width 1)
 		(layer "B.Cu")
@@
 	)
 	(segment
-		(start 213.36 114.3)
-		(end 212.09 115.57)
+		(start 218.44 82.09)
+		(end 220.44 82.09)
 		(width 1)
 		(layer "B.Cu")
@@
 	)
 	(segment
-		(start 207.01 123.19)
-		(end 187.325 123.19)
+		(start 210.82 57.15)
+		(end 179.07 57.15)
 		(width 1)
 		(layer "B.Cu")
@@
 	)
 	(segment
-		(start 142.1 125.73)
-		(end 143.37 124.46)
+		(start 221.19 82.12)
+		(end 221.19 67.52)
+		(width 1)
+		(layer "B.Cu")
+		(net 7)
+	)
+	(segment
+		(start 220.83 82.48)
+		(end 221.19 82.84)
 		(width 1)
 		(layer "B.Cu")
@@
 	)
 	(segment
-		(start 213.36 82.55)
-		(end 213.36 114.3)
+		(start 207.01 123.19)
+		(end 187.325 123.19)
+		(width 1)
+		(layer "B.Cu")
+		(net 7)
+	)
+	(segment
+		(start 142.1 125.73)
+		(end 143.37 124.46)
 		(width 1)
 		(layer "B.Cu")
@@
 	)
 	(segment
-		(start 185.020787 135)
-		(end 201.16 135)
+		(start 182.245 133.565)
+		(end 183.68 135)
 		(width 1)
 		(layer "B.Cu")
@@
 	)
 	(segment
-		(start 182.245 130.81)
-		(end 182.245 132.224213)
+		(start 201.16 135)
+		(end 205.62 130.54)
 		(width 1)
 		(layer "B.Cu")
@@
 	)
 	(segment
-		(start 201.16 135)
-		(end 205.62 130.54)
+		(start 183.68 135)
+		(end 201.16 135)
 		(width 1)
 		(layer "B.Cu")
@@
 	)
 	(segment
-		(start 182.245 132.224213)
-		(end 185.020787 135)
+		(start 182.245 130.81)
+		(end 182.245 133.565)
 		(width 1)
 		(layer "B.Cu")
@@
 	)
 	(segment
-		(start 209.545 68.585)
-		(end 207.615 68.585)
+		(start 209.55 68.58)
+		(end 210.82 68.58)
 		(width 1)
 		(layer "B.Cu")
@@
 	)
 	(segment
-		(start 210.82 74.93)
-		(end 210.82 68.58)
-		(width 1)
-		(layer "B.Cu")
-		(net 50)
-	)
-	(segment
-		(start 209.55 68.58)
-		(end 209.545 68.585)
+		(start 207.615 68.585)
+		(end 207.615 63.275)
 		(width 1)
 		(layer "B.Cu")
@@
 	)
 	(segment
-		(start 207.615 68.585)
-		(end 207.615 63.275)
+		(start 210.82 81.57)
+		(end 213.34 84.09)
 		(width 1)
 		(layer "B.Cu")
@@
 	)
 	(segment
-		(start 209.55 84.55)
-		(end 204.47 84.55)
+		(start 213.34 84.09)
+		(end 218.44 84.09)
 		(width 1)
 		(layer "B.Cu")
@@
 	)
 	(segment
-		(start 204.47 84.55)
-		(end 204.47 74.93)
+		(start 209.545 68.585)
+		(end 209.55 68.58)
 		(width 1)
 		(layer "B.Cu")
@@
 	(segment
 		(start 210.82 68.58)
-		(end 209.55 68.58)
+		(end 210.82 81.57)
 		(width 1)
 		(layer "B.Cu")
@@
 	)
 	(segment
-		(start 204.47 74.93)
-		(end 210.82 74.93)
+		(start 207.615 68.585)
+		(end 209.545 68.585)
 		(width 1)
 		(layer "B.Cu")
@@
 	)
 	(segment
+		(start 189.98 131.781657)
+		(end 188.371657 133.39)
+		(width 1)
+		(layer "B.Cu")
+		(net 56)
+	)
+	(segment
+		(start 185.05 133.39)
+		(end 184.785 133.125)
+		(width 1)
+		(layer "B.Cu")
+		(net 56)
+	)
+	(segment
 		(start 188.845 71.505)
 		(end 189.23 71.12)
@@
 	)
 	(segment
+		(start 189.98 127.029213)
+		(end 189.98 131.781657)
+		(width 1)
+		(layer "B.Cu")
+		(net 56)
+	)
+	(segment
 		(start 185.910787 102.87)
 		(end 187.43637 102.87)
@@
 	)
 	(segment
+		(start 214 125.46)
+		(end 213.54 125)
+		(width 1)
+		(layer "B.Cu")
+		(net 56)
+	)
+	(segment
 		(start 185.42 109.25)
 		(end 185.39 109.22)
@@
 	)
 	(segment
-		(start 189.325 131.638428)
-		(end 188.153428 132.81)
+		(start 213.54 125)
+		(end 192.009213 125)
 		(width 1)
 		(layer "B.Cu")
@@
 	)
 	(segment
-		(start 185.370787 132.81)
-		(end 184.785 132.224213)
-		(width 1)
-		(layer "B.Cu")
-		(net 56)
-	)
-	(segment
 		(start 124.6 91.76)
 		(end 124.6 117.63)
@@
 	)
 	(segment
-		(start 220.71 41.01)
-		(end 220.3 40.6)
+		(start 184.785 133.125)
+		(end 184.785 130.81)
 		(width 1)
 		(layer "B.Cu")
@@
 	)
 	(segment
-		(start 184.785 132.224213)
-		(end 184.785 130.81)
+		(start 192.009213 125)
+		(end 189.98 127.029213)
 		(width 1)
 		(layer "B.Cu")
@@
 	)
 	(segment
-		(start 189.325 127.684213)
-		(end 189.325 131.638428)
+		(start 220.71 41.01)
+		(end 220.3 40.6)
 		(width 1)
 		(layer "B.Cu")
@@
 	)
 	(segment
-		(start 213.54 125)
-		(end 192.009213 125)
+		(start 173.77 52.07)
+		(end 172.085 52.07)
 		(width 1)
 		(layer "B.Cu")
@@
 	)
 	(segment
-		(start 173.77 52.07)
-		(end 172.085 52.07)
+		(start 188.371657 133.39)
+		(end 185.05 133.39)
 		(width 1)
 		(layer "B.Cu")
@@
 		(width 1)
 		(layer "B.Cu")
-		(net 56)
-	)
-	(segment
-		(start 192.009213 125)
-		(end 189.325 127.684213)
-		(width 1)
-		(layer "B.Cu")
-		(net 56)
-	)
-	(segment
-		(start 214 125.46)
-		(end 213.54 125)
-		(width 1)
-		(layer "B.Cu")
-		(net 56)
-	)
-	(segment
-		(start 188.153428 132.81)
-		(end 185.370787 132.81)
-		(width 1)
-		(layer "B.Cu")
