File: PCB/Ambush/V1/V1.kicad_sch (KiCad schematic)
At the start: 7 parts, among them J1 Pines Motores, J2 Screw_Terminal_01x02, SW1 SW ON/OFF, U2 ESP32-Devkit-V1

Commit message: PCB Con testpoint
Parts:
- added J10, J3, J4, J5, J6, J7, J8, J9: Conn_01x01_Pin, Connector_PinHeader_2.54mm:PinHeader_1x01_P2.54mm_Vertical, symbol Connector:Conn_01x01_Pin
Connections:
- net +5V: now also J9.1 (Pin_1)
- net AIN1 MONSTER SHIELD: now also J6.1 (Pin_1)
- net AIN2 MONSTER SHIELD: now also J7.1 (Pin_1)
- net BIN 1 MONSTER SHIELD: now also J3.1 (Pin_1)
- net BIN 2 MONSTER SHIELD: now also J8.1 (Pin_1)
- net GND: now also J10.1 (Pin_1)
- net PWM A MONSTER SHIELD: now also J4.1 (Pin_1)
- net PWM B MONSTER SHIELD: now also J5.1 (Pin_1)
Other:
- note added: "TEST POINT"
